File: V2/Hardware/breakout/breakout.kicad_pcb (KiCad board)
At the start: 2 copper layers, 8 parts, among them J0 Flat_7seg_F, J1 Conn_D, J2 Conn_C, J3 Conn_E, J4 Conn_B, J5 Conn_F, J6 Conn_A, J7 Conn_G

Commit message: Export -pcbs
Routing:
- net /+12V: track 146.8 -> 180.8 mm
- net (no net): vias 0 -> 4
Other:
- board text added: "33mm"
- board text added: "56mm"

Commit message: Make more precise plots
Routing:
- net (no net): track 0.00 -> 4.00 mm
Changed lines of the file:
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@@
   (general
     (thickness 1.6)
-    (drawings 10)
-    (tracks 88)
+    (drawings 16)
+    (tracks 96)
     (zones 0)
     (modules 8)
@@
   )
   (setup
-    (last_trace_width 1.5)
+    (last_trace_width 0.25)
     (user_trace_width 1.5)
     (user_trace_width 2)
@@
     (visible_elements FFFFFF7F)
     (pcbplotparams
-      (layerselection 0x01800_fffffffe)
+      (layerselection 0x00800_fffffffe)
       (usegerberextensions false)
       (usegerberattributes true)
       (usegerberadvancedattributes true)
       (creategerberjobfile true)
-      (excludeedgelayer true)
+      (excludeedgelayer false)
       (linewidth 0.100000)
       (plotframeref false)
@@
       (plotvalue false)
       (plotinvisibletext false)
-      (padsonsilk false)
+      (padsonsilk true)
       (subtractmaskfromsilk false)
       (outputformat 5)
@@
     )
   )
+  (gr_circle (center 136 67) (end 137 66) (layer Eco2.User) (width 0.25))
+  (gr_circle (center 136 86) (end 137 85) (layer Eco2.User) (width 0.25))
+  (gr_circle (center 180 86) (end 181 85) (layer Eco2.User) (width 0.25))
+  (gr_circle (center 180 67) (end 181 68) (layer Eco2.User) (width 0.25))
+  (gr_line (start 145 85) (end 143 85) (layer Eco2.User) (width 0.25))
+  (gr_line (start 144 84) (end 144 86) (layer Eco2.User) (width 0.25))
   (gr_text 33mm (at 183 82) (layer Eco2.User)
     (effects (font (size 1 1) (thickness 0.15)))
@@
   (via (at 136 86) (size 0.8) (drill 0.4) (layers F.Cu B.Cu) (net 0))
   (via (at 136 67) (size 0.8) (drill 0.4) (layers F.Cu B.Cu) (net 0))
-  (segment (start 160 62) (end 160 65) (width 1.5) (layer B.Cu) (net 1))
+  (segment (start 144 84) (end 144 86) (width 0.25) (layer B.Cu) (net 0))
+  (segment (start 143 85) (end 145 85) (width 0.25) (layer B.Cu) (net 0))
   (segment (start 160 65) (end 165 70) (width 1.5) (layer B.Cu) (net 1))
   (segment (start 165 70) (end 165 76) (width 1.5) (layer B.Cu) (net 1))
+  (segment (start 160 62) (end 160 63) (width 2) (layer B.Cu) (net 1))
+  (segment (start 160 63) (end 160 65) (width 1.5) (layer B.Cu) (net 1))
   (segment (start 166.46 78.54) (end 168 77) (width 1.5) (layer B.Cu) (net 2))
-  (segment (start 168 77) (end 168 62) (width 1.5) (layer B.Cu) (net 2))
   (segment (start 165 78.54) (end 166.46 78.54) (width 1.5) (layer B.Cu) (net 2))
+  (segment (start 168 62) (end 168 63) (width 2) (layer B.Cu) (net 2))
+  (segment (start 168 77) (end 168 63) (width 1.5) (layer B.Cu) (net 2))
   (segment (start 162.46 71.46) (end 158 67) (width 1.5) (layer B.Cu) (net 3))
   (segment (start 158 67) (end 154 67) (width 1.5) (layer B.Cu) (net 3))
   (segment (start 154 67) (end 152 65) (width 1.5) (layer B.Cu) (net 3))
-  (segment (start 152 65) (end 152 62) (width 1.5) (layer B.Cu) (net 3))
   (segment (start 162.46 76) (end 162.46 71.46) (width 1.5) (layer B.Cu) (net 3))
+  (segment (start 152 62) (end 152 63) (width 2) (layer B.Cu) (net 3))
+  (segment (start 152 65) (end 152 63) (width 1.5) (layer B.Cu) (net 3))
   (segment (start 162.46 79.742081) (end 163.717919 81) (width 1.5) (layer B.Cu) (net 4))
   (segment (start 163.717919 81) (end 168 81) (width 1.5) (layer B.Cu) (net 4))
   (segment (start 168 81) (end 176 73) (width 1.5) (layer B.Cu) (net 4))
-  (segment (start 176 73) (end 176 62) (width 1.5) (layer B.Cu) (net 4))
   (segment (start 162.46 78.54) (end 162.46 79.742081) (width 1.5) (layer B.Cu) (net 4))
+  (segment (start 176 62) (end 176 63) (width 2) (layer B.Cu) (net 4))
+  (segment (start 176 73) (end 176 63) (width 1.5) (layer B.Cu) (net 4))
   (segment (start 151 70) (end 157 70) (width 1.5) (layer B.Cu) (net 5))
   (segment (start 157 70) (end 159.92 72.92) (width 1.5) (layer B.Cu) (net 5))
   (segment (start 144 63) (end 151 70) (width 1.5) (layer B.Cu) (net 5))
-  (segment (start 144 62) (end 144 63) (width 1.5) (layer B.Cu) (net 5))
   (segment (start 159.92 72.92) (end 159.92 76) (width 1.5) (layer B.Cu) (net 5))
+  (segment (start 144 62) (end 144 63) (width 2) (layer B.Cu) (net 5))
   (segment (start 171 84) (end 183 72) (width 1.5) (layer B.Cu) (net 6))
   (segment (start 159.92 80.92) (end 163 84) (width 1.5) (layer B.Cu) (net 6))
   (segment (start 163 84) (end 171 84) (width 1.5) (layer B.Cu) (net 6))
-  (segment (start 183 72) (end 183 62) (width 1.5) (layer B.Cu) (net 6))
   (segment (start 159.92 78.54) (end 159.92 80.92) (width 1.5) (layer B.Cu) (net 6))
+  (segment (start 183 62) (end 183 63) (width 2) (layer B.Cu) (net 6))
+  (segment (start 183 72) (end 183 63) (width 1.5) (layer B.Cu) (net 6))
   (segment (start 147 73) (end 156 73) (width 1.5) (layer B.Cu) (net 7))
   (segment (start 156 73) (end 157.38 74.38) (width 1.5) (layer B.Cu) (net 7))
-  (segment (start 136 62) (end 147 73) (width 1.5) (layer B.Cu) (net 7))
   (segment (start 157.38 74.38) (end 157.38 76) (width 1.5) (layer B.Cu) (net 7))
+  (segment (start 136 62) (end 137 63) (width 2) (layer B.Cu) (net 7))
+  (segment (start 137 63) (end 147 73) (width 1.5) (layer B.Cu) (net 7))
   (segment (start 154.84 76) (end 154.84 78.54) (width 1.5) (layer B.Cu) (net 8))
   (segment (start 141.46 62) (end 141.46 59.54) (width 1.5) (layer B.Cu) (net 8))
