File: V2/Hardware/controller/controller.sch (KiCad schematic (older format))
At the start: 52 parts, among them J0 Molex_PSU_F, J2 Flat_7seg_F, J3 Rpi_DATA_F_3.3V, Q0 BD139-16, Q1 BD139-16, Q2 BD139-16, Q3 BD139-16, Q4 BD139-16, Q5 BD139-16, Q6 BD139-16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

Commit message: revision 2 boards
Parts:
- removed J3: Rpi_DATA_F_3.3V, Connector_PinHeader_2.54mm:PinHeader_2x03_P2.54mm_Horizontal, symbol Connector_Generic:Conn_02x03_Counter_Clockwise
- added J3: RPI_DATA_3.3V, Connector_IDC:IDC-Header_2x05-1MP_P2.54mm_Latch_Vertical, symbol Connector_Generic:Conn_02x05_Odd_Even
- J0: value Molex_PSU_F -> Molex_PSU; footprint PSU:conn_hdd_15-24-4441 -> KicadLib:conn_hdd_15-24-4449
- J2: value Flat_7seg_F -> 7SEG_12V; footprint Connector_PinHeader_2.54mm:PinHeader_2x05_P2.54mm_Horizontal -> Connector_IDC:IDC-Header_2x05-1MP_P2.54mm_Latch_Vertical
Connections:
- net BIT_A: now also J3.1 (Pin_1)
- net BIT_B: now also J3.3 (Pin_3)
- net BIT_C: now also J3.5 (Pin_5)
- net BIT_D: now also J3.7 (Pin_7)
- net Earth: now also J3.10 (Pin_10), J3.2 (Pin_2), J3.4 (Pin_4), J3.6 (Pin_6), J3.8 (Pin_8), J3.9 (Pin_9)
- no-connect marks 7 -> 6
Other:
- moved on the sheet: D4, D5, R11, R12
Changed lines of the file:
@@
 L Device:R R12
 U 1 1 5EB47108
-P 3850 4350
-F 0 "R12" H 3920 4396 50  0000 L CNN
-F 1 "1k5" H 3920 4305 50  0000 L CNN
-F 2 "Resistor_THT:R_Axial_DIN0207_L6.3mm_D2.5mm_P10.16mm_Horizontal" V 3780 4350 50  0001 C CNN
-F 3 "~" H 3850 4350 50  0001 C CNN
-	1    3850 4350
+P 3300 4350
+F 0 "R12" H 3370 4396 50  0000 L CNN
+F 1 "1k5" H 3370 4305 50  0000 L CNN
+F 2 "Resistor_THT:R_Axial_DIN0207_L6.3mm_D2.5mm_P10.16mm_Horizontal" V 3230 4350 50  0001 C CNN
+F 3 "~" H 3300 4350 50  0001 C CNN
+	1    3300 4350
 	-1   0    0    1
 $EndComp
-Text Label 3600 2750 0    50   ~ 0
+Text Label 3000 3450 2    50   ~ 0
 BIT_B
 $Comp
@@
 P 700 1550
 F 0 "J0" H 618 1125 50  0000 C CNN
-F 1 "Molex_PSU_F" H 618 1216 50  0000 C CNN
-F 2 "PSU:conn_hdd_15-24-4441" H 700 1550 50  0001 C CNN
+F 1 "Molex_PSU" H 618 1216 50  0000 C CNN
+F 2 "KicadLib:conn_hdd_15-24-4449" H 700 1550 50  0001 C CNN
 F 3 "~" H 700 1550 50  0001 C CNN
 	1    700  1550
@@
 P 10200 1350
 F 0 "J2" H 10250 1750 50  0000 C CNN
-F 1 "Flat_7seg_F" H 10250 1650 50  0000 C CNN
-F 2 "Connector_PinHeader_2.54mm:PinHeader_2x05_P2.54mm_Horizontal" H 10200 1350 50  0001 C CNN
+F 1 "7SEG_12V" H 10250 1650 50  0000 C CNN
+F 2 "Connector_IDC:IDC-Header_2x05-1MP_P2.54mm_Latch_Vertical" H 10200 1350 50  0001 C CNN
 F 3 "~" H 10200 1350 50  0001 C CNN
 	1    10200 1350
@@
 L Device:R R11
 U 1 1 5EB45F1E
-P 3250 4350
-F 0 "R11" H 3320 4396 50  0000 L CNN
-F 1 "1k5" H 3320 4305 50  0000 L CNN
-F 2 "Resistor_THT:R_Axial_DIN0207_L6.3mm_D2.5mm_P10.16mm_Horizontal" V 3180 4350 50  0001 C CNN
-F 3 "~" H 3250 4350 50  0001 C CNN
-	1    3250 4350
+P 3000 4350
+F 0 "R11" H 3070 4396 50  0000 L CNN
+F 1 "1k5" H 3070 4305 50  0000 L CNN
+F 2 "Resistor_THT:R_Axial_DIN0207_L6.3mm_D2.5mm_P10.16mm_Horizontal" V 2930 4350 50  0001 C CNN
+F 3 "~" H 3000 4350 50  0001 C CNN
+	1    3000 4350
 	-1   0    0    1
 $EndComp
@@
 L Device:LED D4
 U 1 1 5FC9598B
-P 3250 4650
-F 0 "D4" V 3289 4532 50  0000 R CNN
-F 1 "LED_2V_20mA" V 3198 4532 50  0000 R CNN
-F 2 "LED_THT:LED_D5.0mm" H 3250 4650 50  0001 C CNN
-F 3 "~" H 3250 4650 50  0001 C CNN
-	1    3250 4650
+P 3000 4650
+F 0 "D4" V 3039 4532 50  0000 R CNN
+F 1 "LED_2V_20mA" V 2948 4532 50  0000 R CNN
+F 2 "LED_THT:LED_D5.0mm" H 3000 4650 50  0001 C CNN
+F 3 "~" H 3000 4650 50  0001 C CNN
+	1    3000 4650
 	0    -1   -1   0
 $EndComp
@@
 L Device:LED D5
 U 1 1 5FC961FF
-P 3850 4650
-F 0 "D5" V 3889 4532 50  0000 R CNN
-F 1 "LED_2V_20mA" V 3798 4532 50  0000 R CNN
-F 2 "LED_THT:LED_D5.0mm" H 3850 4650 50  0001 C CNN
-F 3 "~" H 3850 4650 50  0001 C CNN
-	1    3850 4650
+P 3300 4650
+F 0 "D5" V 3339 4532 50  0000 R CNN
+F 1 "LED_2V_20mA" V 3248 4532 50  0000 R CNN
+F 2 "LED_THT:LED_D5.0mm" H 3300 4650 50  0001 C CNN
+F 3 "~" H 3300 4650 50  0001 C CNN
+	1    3300 4650
 	0    -1   -1   0
 $EndComp
@@
 Connection ~ 2700 4900
 Wire Wire Line
-	2700 4900 3250 4900
-Wire Wire Line
-	3250 4800 3250 4900
-Connection ~ 3250 4900
-Wire Wire Line
-	3250 4900 3850 4900
-Wire Wire Line
-	3850 4800 3850 4900
-Connection ~ 3850 4900
+	2700 4900 3000 4900
+Wire Wire Line
+	3000 4800 3000 4900
+Connection ~ 3000 4900
+Wire Wire Line
+	3000 4900 3300 4900
+Wire Wire Line
+	3300 4800 3300 4900
+Connection ~ 3300 4900
 Wire Wire Line
 	2400 3850 5450 3850
@@
 	2700 3950 2700 4200
 Wire Wire Line
-	3250 4050 5750 4050
-Wire Wire Line
-	3250 4050 3250 4200
+	3000 4050 5750 4050
+Wire Wire Line
+	3000 4050 3000 4200
 Wire Wire Line
 	5450 2950 5100 2950
@@
 Text Notes 5250 2800 0    50   ~ 0
 1 pin - 4.5V 3mA, 21mA over all pins \nMax per pin: 20mA\nMax over all pins: 60mA
-Text Notes 2400 2650 0    50   ~ 0
+Text Notes 2400 2950 0    50   ~ 0
 3.3V 800uA
 Text Notes 3900 1350 0    50   ~ 0
@@
 Wire Wire Line
 	9800 1700 9800 4350
-Wire Wire Line
-	2700 2850 2700 3950
-Wire Wire Line
-	3700 2750 3600 2750
-Text Label 3100 2650 2    50   ~ 0
+Text Label 2400 3450 2    50   ~ 0
 BIT_D
-Text Label 3100 2850 2    50   ~ 0
+Text Label 2700 3450 2    50   ~ 0
 BIT_C
-Text Label 3600 2650 0    50   ~ 0
+Text Label 3300 3450 2    50   ~ 0
 BIT_A
-$Comp
-L Connector_Generic:Conn_02x03_Counter_Clockwise J3
-U 1 1 5EA33B7C
-P 3300 2750
-F 0 "J3" H 3350 3067 50  0000 C CNN
-F 1 "Rpi_DATA_F_3.3V" H 3350 2976 50  0000 C CNN
-F 2 "Connector_PinHeader_2.54mm:PinHeader_2x03_P2.54mm_Horizontal" H 3300 2750 50  0001 C CNN
-F 3 "~" H 3300 2750 50  0001 C CNN
-	1    3300 2750
-	1    0    0    -1
-$EndComp
-Wire Wire Line
-	3850 4150 5900 4150
-Wire Wire Line
-	3850 4150 3850 4200
-Connection ~ 3850 4150
-Wire Wire Line
-	3850 4900 4500 4900
-Wire Wire Line
-	3850 2650 3600 2650
-Wire Wire Line
-	3850 2650 3850 4150
-NoConn ~ 3100 2750
-Wire Wire Line
-	2700 2850 3100 2850
-Wire Wire Line
-	2400 2650 3100 2650
-Wire Wire Line
-	2400 2650 2400 3850
-Wire Wire Line
-	3700 2750 3700 3250
-Wire Wire Line
-	3700 3250 3250 3250
-Wire Wire Line
-	3250 3250 3250 4050
-Connection ~ 3250 4050
-Wire Wire Line
-	3100 2850 3100 3000
-Wire Wire Line
-	3100 3000 3600 3000
-Wire Wire Line
-	3600 3000 3600 2850
-Connection ~ 3100 2850
+Wire Wire Line
+	3300 4150 5900 4150
+Wire Wire Line
+	3300 4150 3300 4200
+Connection ~ 3300 4150
+Wire Wire Line
+	3300 4900 4500 4900
+Wire Wire Line
+	2400 2950 2400 3850
+Connection ~ 3000 4050
 Wire Wire Line
 	10750 900  10750 1150
@@
 Wire Wire Line
 	2250 2150 2800 2150
+$Comp
+L Connector_Generic:Conn_02x05_Odd_Even J3
+U 1 1 60C34227
+P 3550 2850
+F 0 "J3" H 3550 3250 50  0000 C CNN
+F 1 "RPI_DATA_3.3V" H 3550 3150 50  0000 C CNN
+F 2 "Connector_IDC:IDC-Header_2x05-1MP_P2.54mm_Latch_Vertical" H 3550 2850 50  0001 C CNN
+F 3 "~" H 3550 2850 50  0001 C CNN
+	1    3550 2850
+	1    0    0    -1
+$EndComp
+Wire Wire Line
+	3700 2150 3850 2150
+Wire Wire Line
+	3850 2150 3850 2650
+Connection ~ 3700 2150
+Wire Wire Line
+	3850 2650 3850 2750
+Connection ~ 3850 2650
+Wire Wire Line
+	3850 2750 3850 2850
+Connection ~ 3850 2750
+Wire Wire Line
+	3850 2850 3850 2950
+Connection ~ 3850 2850
+Wire Wire Line
+	2400 2950 3350 2950
+Wire Wire Line
+	2700 2850 3350 2850
+Wire Wire Line
+	2700 2850 2700 3950
+Wire Wire Line
+	3000 2750 3350 2750
+Wire Wire Line
+	3000 2750 3000 4050
+Wire Wire Line
+	3300 2650 3350 2650
+Wire Wire Line
+	3300 2650 3300 4150
+Wire Wire Line
+	3850 3050 3850 2950
+Connection ~ 3850 2950
+Wire Wire Line
+	3350 3050 3350 3150
+Wire Wire Line
+	3350 3150 3850 3150
+Wire Wire Line
+	3850 3150 3850 3050
+Connection ~ 3850 3050
 $EndSCHEMATC
