File: V2/Hardware/burner/burner.kicad_pcb (KiCad board)
At the start: 2 copper layers, 2 parts, among them J1 ISP connector, U1 ATtiny2313-20PU

Commit message: revision 2 boards
Other:
- board text added: "23 mm"
- board text added: "41 mm"
- board text removed: "23mm"
- board text removed: "41mm"
Changed lines of the file:
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@@
     (visible_elements FFFFFF7F)
     (pcbplotparams
-      (layerselection 0x010fc_ffffffff)
+      (layerselection 0x00840_fffffffe)
       (usegerberextensions false)
       (usegerberattributes true)
@@
       (padsonsilk false)
       (subtractmaskfromsilk false)
-      (outputformat 1)
+      (outputformat 3)
       (mirror false)
       (drillshape 1)
       (scaleselection 1)
-      (outputdirectory ""))
+      (outputdirectory "DXF/"))
   )
   (net 0 "")
@@
     )
   )
-  (target plus (at 129 117) (size 5) (width 0.05) (layer Edge.Cuts))
-  (target plus (at 129 117) (size 5) (width 0.05) (layer Edge.Cuts))
-  (gr_text 23mm (at 128 120) (layer Eco2.User)
+  (target plus (at 130 117) (size 5) (width 0.05) (layer Edge.Cuts))
+  (target plus (at 130 117) (size 5) (width 0.05) (layer Edge.Cuts))
+  (gr_text "23 mm" (at 128 120) (layer Eco2.User)
     (effects (font (size 1 1) (thickness 0.15)))
   )
-  (gr_text 41mm (at 126 115 90) (layer Eco2.User)
+  (gr_text "41 mm" (at 126 115 90) (layer Eco2.User)
     (effects (font (size 1 1) (thickness 0.15)))
   )
